File: Tiny handheld.kicad_pcb (KiCad board)
At the start: 2 copper layers, 34.3 x 58.4 mm, 38 parts, among them J1 Conn_01x04_Female, J3 TYPE-C-31-M-12, U1 ATtiny85-20P, U2 ATtiny85-20M, U3 EEPROM-I2CEIAJ

Commit message: updated schematic (nothing special)
Other:
- board text added: "Designed by: Casper R. Tak"
- board text added: "Tiny Handheld"
- board text added: "remove battery when uploading program/games"
- board text removed: "Tiny Handheld Casper R. Tak"
Changed lines of the file:
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@@
     (fp_arc (start 7.84 -8) (mid 9.50994 -5.917963) (end 10.64 -3.5) (layer "B.SilkS") (width 0.127))
     (fp_arc (start 10.64 3.5) (mid 9.509972 5.917983) (end 7.84 8) (layer "B.SilkS") (width 0.127))
-    (fp_arc (start -10.64 -3.5) (mid -9.509973 -5.917983) (end -7.84 -8) (layer "B.SilkS") (width 0.127))
+    (fp_arc (start -10.64 -3.5) (mid -9.509972 -5.917982) (end -7.84 -8) (layer "B.SilkS") (width 0.127))
     (fp_line (start -14.55 -8.25) (end -14.55 8.25) (layer "B.CrtYd") (width 0.05))
     (fp_line (start 14.55 8.25) (end 14.55 -8.25) (layer "B.CrtYd") (width 0.05))
@@
     (fp_line (start 14.3 -3.5) (end 10.64 -3.5) (layer "B.Fab") (width 0.127))
     (fp_arc (start 7.84 -8) (mid 9.50994 -5.917963) (end 10.64 -3.5) (layer "B.Fab") (width 0.127))
-    (fp_arc (start -10.64 -3.5) (mid -9.509973 -5.917983) (end -7.84 -8) (layer "B.Fab") (width 0.127))
+    (fp_arc (start -10.64 -3.5) (mid -9.509972 -5.917982) (end -7.84 -8) (layer "B.Fab") (width 0.127))
     (fp_arc (start -7.84 8) (mid -9.509941 5.917963) (end -10.64 3.5) (layer "B.Fab") (width 0.127))
     (fp_arc (start 10.64 3.5) (mid 9.509972 5.917983) (end 7.84 8) (layer "B.Fab") (width 0.127))
@@
   (gr_line (start 153.67 72.39) (end 180.34 72.39) (layer "Edge.Cuts") (width 0.1))
   (gr_line (start 180.34 130.81) (end 153.67 130.81) (layer "Edge.Cuts") (width 0.1))
-  (gr_text "CR2032 Battery" (at 159.004 89.916) (layer "B.SilkS")
-    (effects (font (size 1 1) (thickness 0.15)) (justify mirror))
-  )
   (gr_text "5V usb" (at 167.64 126.492) (layer "B.SilkS")
     (effects (font (size 1 1) (thickness 0.15)) (justify mirror))
@@
     (effects (font (size 0.5 0.5) (thickness 0.125)) (justify mirror))
   )
-  (gr_text "Tiny Handheld\nCasper R. Tak" (at 178.308 123.952) (layer "B.SilkS")
+  (gr_text "Designed by:\nCasper R. Tak" (at 178.308 123.952) (layer "B.SilkS")
     (effects (font (size 1 1) (thickness 0.15)) (justify mirror))
   )
+  (gr_text "CR2032 Battery" (at 158.242 103.3272) (layer "B.SilkS")
+    (effects (font (size 1 1) (thickness 0.15)) (justify mirror))
+  )
+  (gr_text "remove battery \nwhen uploading \nprogram/games" (at 156.1592 119.4816) (layer "B.SilkS")
+    (effects (font (size 1 1) (thickness 0.15)) (justify mirror))
+  )
+  (gr_text "Tiny Handheld" (at 178.435 120.015) (layer "F.SilkS")
+    (effects (font (size 1 1) (thickness 0.15)))
+  )
   (via (at 153.67 76.2) (size 5) (drill 4) (layers "F.Cu" "B.Cu") (free) (net 0))

Commit message: started routing
Connections:
- U1 pad 1: Net-(U1-Pad1) -> PB5/RES
- U1 pad 2: Net-(U1-Pad2) -> PB3
- U1 pad 3: Net-(U1-Pad3) -> PB4
- U1 pad 5: Net-(U1-Pad5) -> PB0/SDA/MOSI
- U1 pad 6: Net-(U1-Pad6) -> PB1/MISO
- U1 pad 7: Net-(U1-Pad7) -> PB2/SCL/SCK
- U2 pad 1: Net-(U1-Pad1) -> PB5/RES
- U2 pad 11: Net-(U1-Pad5) -> PB0/SDA/MOSI
- U2 pad 12: Net-(U1-Pad6) -> PB1/MISO
- U2 pad 14: Net-(U1-Pad7) -> PB2/SCL/SCK
- U2 pad 2: Net-(U1-Pad2) -> PB3
- U2 pad 5: Net-(U1-Pad3) -> PB4
Routing:
- net PB1/MISO: track 0.00 -> 27.4 mm
- net PB3: track 0.00 -> 19.5 mm
- net Net-(JP1-Pad1): track 0.00 -> 8.92 mm
Other:
- board text added: "+"
- board text added: "0.96 inch i2c oled screen"
- board text added: "5V usb External power"
- board text added: "GND"
- board text added: "PB0 SDA"
- board text added: "PB2 SCL"
- board text added: "SCL"
- board text added: "SDA"
- board text added: "Tiny Handheld V1.0"
- board text added: "VCC"
- board text removed: "5V usb"
- board text removed: "Tiny Handheld"
- board text removed: "remove battery when uploading program/games"
