File: Tiny handheld.kicad_sch (KiCad schematic)
At the start: 41 parts, among them IC1 BQ21040DBVR, J1 VDisplay/prog1, J2 HDisplay/prog, J3 USB_C_Receptacle_USB2.0, U1 ATtiny85-20P, U2 ATtiny85-20S

Commit message: cleanup
Parts:
- renumbered 5V to 5V1, GND to GND1, en-charge to en-charge1
Changed lines of the file:
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@@
   (symbol (lib_id "Connector:TestPoint") (at 57.15 104.775 0) (unit 1)
     (in_bom yes) (on_board yes)
-    (property "Reference" "5V" (id 0) (at 59.69 100.2029 0)
+    (property "Reference" "5V1" (id 0) (at 59.69 100.2029 0)
       (effects (font (size 1.27 1.27)) (justify left))
     )
@@
   (symbol (lib_id "Connector:TestPoint") (at 43.815 137.16 180) (unit 1)
     (in_bom yes) (on_board yes) (fields_autoplaced)
-    (property "Reference" "GND" (id 0) (at 45.72 139.1919 0)
+    (property "Reference" "GND1" (id 0) (at 45.72 139.1919 0)
       (effects (font (size 1.27 1.27)) (justify right))
     )
@@
   (symbol (lib_id "Jumper:Jumper_2_Open") (at 140.335 122.555 0) (unit 1)
     (in_bom yes) (on_board yes) (fields_autoplaced)
-    (property "Reference" "en-charge" (id 0) (at 140.335 115.57 0))
+    (property "Reference" "en-charge1" (id 0) (at 140.335 115.57 0))
     (property "Value" "Jumper_2_Open" (id 1) (at 140.335 118.11 0))
     (property "Footprint" "Jumper:SolderJumper-2_P1.3mm_Open_RoundedPad1.0x1.5mm" (id 2) (at 140.335 122.555 0)
@@
     )
     (path "/340146ae-1dcd-4cc9-b1a4-794b73097a69"
-      (reference "5V") (unit 1) (value "5V") (footprint "TestPoint:TestPoint_Pad_1.0x1.0mm")
+      (reference "5V1") (unit 1) (value "5V") (footprint "TestPoint:TestPoint_Pad_1.0x1.0mm")
     )
     (path "/d87d81d6-a9f7-455a-b1d8-8ff0988a0a64"
@@
     )
     (path "/42350c44-064d-4037-affd-69bc19043671"
-      (reference "GND") (unit 1) (value "GND") (footprint "TestPoint:TestPoint_Pad_1.0x1.0mm")
+      (reference "GND1") (unit 1) (value "GND") (footprint "TestPoint:TestPoint_Pad_1.0x1.0mm")
     )
     (path "/a18d266d-c0d2-4b00-9a60-ec95f250657b"
@@
     )
     (path "/bc823d2e-cd93-4e16-8824-0c0bbb02b3b1"
-      (reference "en-charge") (unit 1) (value "Jumper_2_Open") (footprint "Jumper:SolderJumper-2_P1.3mm_Open_RoundedPad1.0x1.5mm")
-    )
-  )
+      (reference "en-charge1") (unit 1) (value "Jumper_2_Open") (footprint "Jumper:SolderJumper-2_P1.3mm_Open_RoundedPad1.0x1.5mm")
+    )
+  )
