File: Tiny Handheld V2.1/Tiny handheld.kicad_sch (KiCad schematic)
At the start: 41 parts, among them IC1 BQ21040DBVR, J1 VDisplay/prog1, J2 HDisplay/prog, J3 USB_C_Receptacle_USB2.0, U1 ATtiny85-20P, U2 ATtiny85-20S

Commit message: enh v2.1
- new 5 way button footprint (functional)
- larger keyhole
- rewired
Parts:
- removed BT1: BATTERY-6.8MM_SMD, Battery:BatteryHolder_Keystone_3002_1x2032, symbol SparkFun-Batteries:BATTERY-6.8MM_SMD
- added BT1: Battery_Cell, Battery:BatteryHolder_Keystone_3002_1x2032, symbol Device:Battery_Cell
- added H1: MountingHole, MountingHole:MountingHole_3.2mm_M3, symbol Mechanical:MountingHole
- renumbered 5V to 5V1, GND to GND1, en-charge to en-chrg1
Connections:
- net BatOut: now also BT1.1 (+)
- net GND: now also BT1.2 (-)
- net at R3.2: now also S2.UP; no longer S2.A (UP)
- net at R7.2: now also S2.RIGHT; no longer S2.B (RIGHT)
- net at R4.2: now also S2.LEFT; no longer S2.C (LEFT)
- net at R1.2: now also S2.DOWN; no longer S2.D (DOWN)
Changed lines of the file:
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@@
   (no_connect (at 215.9 69.85))
   (no_connect (at 215.9 72.39))
-  (wire (pts (xy 147.32 123.825) (xy 147.32 122.555))
+  (wire (pts (xy 147.32 122.555) (xy 147.32 125.73))
     (stroke (width 0) (type default) (color 0 0 0 0))
   )
@@
     )
     (property "Purpose" "Joystick" (id 5) (at 34.29 73.66 0))
-    (pin "A")
-    (pin "B")
-    (pin "C")
+    (pin "UP")
+    (pin "RIGHT")
+    (pin "LEFT")
     (pin "CTR")
-    (pin "D")
+    (pin "DOWN")
     (pin "GND")
   )
@@
   (symbol (lib_id "Connector:TestPoint") (at 57.15 104.775 0) (unit 1)
     (in_bom yes) (on_board yes)
-    (property "Reference" "5V" (id 0) (at 59.69 100.2029 0)
+    (property "Reference" "5V1" (id 0) (at 59.69 100.2029 0)
       (effects (font (size 1.27 1.27)) (justify left))
     )
@@
     (pin "6")
   )
+  (symbol (lib_id "Device:Battery_Cell") (at 147.32 130.81 0) (unit 1)
+    (in_bom yes) (on_board yes)
+    (property "Reference" "BT1" (id 0) (at 147.955 132.08 0)
+      (effects (font (size 1.27 1.27)) (justify left))
+    )
+    (property "Value" "Battery_Cell" (id 1) (at 150.495 130.0479 0)
+      (effects (font (size 1.27 1.27)) (justify left) hide)
+    )
+    (property "Footprint" "Battery:BatteryHolder_Keystone_3002_1x2032" (id 2) (at 147.32 129.286 90)
+      (effects (font (size 1.27 1.27)) hide)
+    )
+    (property "Datasheet" "~" (id 3) (at 147.32 129.286 90)
+      (effects (font (size 1.27 1.27)) hide)
+    )
+    (pin "1")
+    (pin "2")
+  )
   (symbol (lib_id "Connector:Conn_01x06_Female") (at 255.905 24.765 0) (unit 1)
     (in_bom yes) (on_board yes) (fields_autoplaced)
@@
   (symbol (lib_id "Connector:TestPoint") (at 43.815 137.16 180) (unit 1)
     (in_bom yes) (on_board yes) (fields_autoplaced)
-    (property "Reference" "GND" (id 0) (at 45.72 139.1919 0)
+    (property "Reference" "GND1" (id 0) (at 45.72 139.1919 0)
       (effects (font (size 1.27 1.27)) (justify right))
     )
@@
       (effects (font (size 1.27 1.27)) hide)
     )
-    (property "Datasheet" "https://www.usb.org/sites/default/files/documents/usb_type-c.zip" (id 3) (at 45.085 145.415 0)
+    (property "Datasheet" "file:///C:/Users/crtak/AppData/Local/Temp/Temp1_USBC6P-master.zip/USBC6P-master/Datasheets/USCX-06FX-XXMX-01.pdf" (id 3) (at 45.085 145.415 0)
       (effects (font (size 1.27 1.27)) hide)
     )
@@
     (pin "2")
   )
+  (symbol (lib_id "Mechanical:MountingHole") (at 152.4 145.415 0) (unit 1)
+    (in_bom yes) (on_board yes) (fields_autoplaced)
+    (property "Reference" "H1" (id 0) (at 154.94 144.1449 0)
+      (effects (font (size 1.27 1.27)) (justify left))
+    )
+    (property "Value" "MountingHole" (id 1) (at 154.94 146.6849 0)
+      (effects (font (size 1.27 1.27)) (justify left))
+    )
+    (property "Footprint" "MountingHole:MountingHole_3.2mm_M3" (id 2) (at 152.4 145.415 0)
+      (effects (font (size 1.27 1.27)) hide)
+    )
+    (property "Datasheet" "~" (id 3) (at 152.4 145.415 0)
+      (effects (font (size 1.27 1.27)) hide)
+    )
+  )
   (symbol (lib_id "power:GND") (at 129.54 41.91 0) (unit 1)
     (in_bom yes) (on_board yes) (fields_autoplaced)
@@
   (symbol (lib_id "Jumper:Jumper_2_Open") (at 140.335 122.555 0) (unit 1)
     (in_bom yes) (on_board yes) (fields_autoplaced)
-    (property "Reference" "en-charge" (id 0) (at 140.335 115.57 0))
+    (property "Reference" "en-chrg1" (id 0) (at 140.335 115.57 0))
     (property "Value" "Jumper_2_Open" (id 1) (at 140.335 118.11 0))
     (property "Footprint" "Jumper:SolderJumper-2_P1.3mm_Open_RoundedPad1.0x1.5mm" (id 2) (at 140.335 122.555 0)
@@
     (pin "1")
   )
-  (symbol (lib_id "SparkFun-Batteries:BATTERY-6.8MM_SMD") (at 147.32 128.905 270) (unit 1)
-    (in_bom yes) (on_board yes)
-    (property "Reference" "BT1" (id 0) (at 151.765 130.175 90)
-      (effects (font (size 1.143 1.143)) (justify left))
-    )
-    (property "Value" "BATTERY-6.8MM_SMD" (id 1) (at 152.4 128.905 90)
-      (effects (font (size 1.143 1.143)) (justify left) hide)
-    )
-    (property "Footprint" "Battery:BatteryHolder_Keystone_3002_1x2032" (id 2) (at 153.67 128.905 0)
-      (effects (font (size 0.508 0.508)) hide)
-    )
-    (property "Datasheet" "" (id 3) (at 147.32 128.905 0)
-      (effects (font (size 1.27 1.27)) hide)
-    )
-    (property "Field4" "BATT-13734" (id 4) (at 152.4 132.08 90)
-      (effects (font (size 1.524 1.524)) (justify left) hide)
-    )
-    (property "Purpose" "Rechargeble C2032" (id 5) (at 161.29 127.635 90))
-    (pin "+")
-    (pin "-")
-  )
   (symbol (lib_id "Device:R") (at 117.475 137.795 0) (unit 1)
     (in_bom yes) (on_board yes) (fields_autoplaced)
@@
     (pin "2")
   )
-  (symbol (lib_id "power:GND") (at 147.32 133.985 0) (unit 1)
-    (in_bom yes) (on_board yes) (fields_autoplaced)
-    (property "Reference" "#PWR0106" (id 0) (at 147.32 140.335 0)
-      (effects (font (size 1.27 1.27)) hide)
-    )
-    (property "Value" "GND" (id 1) (at 147.32 139.065 0))
-    (property "Footprint" "" (id 2) (at 147.32 133.985 0)
-      (effects (font (size 1.27 1.27)) hide)
-    )
-    (property "Datasheet" "" (id 3) (at 147.32 133.985 0)
+  (symbol (lib_id "power:GND") (at 147.32 133.35 0) (unit 1)
+    (in_bom yes) (on_board yes) (fields_autoplaced)
+    (property "Reference" "#PWR0106" (id 0) (at 147.32 139.7 0)
+      (effects (font (size 1.27 1.27)) hide)
+    )
+    (property "Value" "GND" (id 1) (at 147.32 138.43 0))
+    (property "Footprint" "" (id 2) (at 147.32 133.35 0)
+      (effects (font (size 1.27 1.27)) hide)
+    )
+    (property "Datasheet" "" (id 3) (at 147.32 133.35 0)
       (effects (font (size 1.27 1.27)) hide)
     )
@@
     )
     (path "/340146ae-1dcd-4cc9-b1a4-794b73097a69"
-      (reference "5V") (unit 1) (value "5V") (footprint "TestPoint:TestPoint_Pad_1.0x1.0mm")
-    )
-    (path "/d87d81d6-a9f7-455a-b1d8-8ff0988a0a64"
-      (reference "BT1") (unit 1) (value "BATTERY-6.8MM_SMD") (footprint "Battery:BatteryHolder_Keystone_3002_1x2032")
+      (reference "5V1") (unit 1) (value "5V") (footprint "TestPoint:TestPoint_Pad_1.0x1.0mm")
+    )
+    (path "/3d59bb4d-036f-4d79-8b19-af756b6e579c"
+      (reference "BT1") (unit 1) (value "Battery_Cell") (footprint "Battery:BatteryHolder_Keystone_3002_1x2032")
     )
     (path "/9a466694-786a-4465-b0d4-e2ee7f1fd8e9"
@@
     )
     (path "/42350c44-064d-4037-affd-69bc19043671"
-      (reference "GND") (unit 1) (value "GND") (footprint "TestPoint:TestPoint_Pad_1.0x1.0mm")
+      (reference "GND1") (unit 1) (value "GND") (footprint "TestPoint:TestPoint_Pad_1.0x1.0mm")
+    )
+    (path "/84ef87af-6f34-4acb-9634-81c71b17a332"
+      (reference "H1") (unit 1) (value "MountingHole") (footprint "MountingHole:MountingHole_3.2mm_M3")
     )
     (path "/a18d266d-c0d2-4b00-9a60-ec95f250657b"
@@
     )
     (path "/bc823d2e-cd93-4e16-8824-0c0bbb02b3b1"
-      (reference "en-charge") (unit 1) (value "Jumper_2_Open") (footprint "Jumper:SolderJumper-2_P1.3mm_Open_RoundedPad1.0x1.5mm")
-    )
-  )
+      (reference "en-chrg1") (unit 1) (value "Jumper_2_Open") (footprint "Jumper:SolderJumper-2_P1.3mm_Open_RoundedPad1.0x1.5mm")
+    )
+  )

Commit message: Improved wiring spacing
Parts:
- en-chrg1: Purpose (none) -> activate charging circuit
Other:
- note added: "Close solder jumper to use charging IC"
Changed lines of the file:
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@@
+    (effects (font (size 1 1)) (justify left bottom))
+  )
+  (text "Close solder jumper \nto use charging IC" (at 148.59 118.11 0)
     (effects (font (size 1 1)) (justify left bottom))
   )
@@
       (effects (font (size 1.27 1.27)) hide)
     )
+    (property "Purpose" "activate charging circuit" (id 4) (at 140.335 122.555 0)
+      (effects (font (size 1.27 1.27)) hide)
+    )

Commit message: cleanup
Changed lines of the file:
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@@
     )
   )
-  (global_label "VCC" (shape input) (at 140.335 56.515 90) (fields_autoplaced)
-    (effects (font (size 1.27 1.27)) (justify left))
-    (property "Intersheet References" "${INTERSHEET_REFS}" (id 0) (at 140.2556 50.4733 90)
-      (effects (font (size 1.27 1.27)) (justify left) hide)
+  (global_label "VCC" (shape input) (at 140.335 56.515 180) (fields_autoplaced)
+    (effects (font (size 1.27 1.27)) (justify right))
+    (property "Intersheet References" "${INTERSHEET_REFS}" (id 0) (at 134.2933 56.5944 0)
+      (effects (font (size 1.27 1.27)) (justify right) hide)
     )
   )

Commit message: added JY JX and JC to schematic
Other:
- note added: "JC"
- note added: "JX"
- note added: "JY"
Changed lines of the file:
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@@
+    (effects (font (size 1.27 1.27)) (justify left bottom))
+  )
+  (text "JY" (at 26.035 39.37 0)
     (effects (font (size 1.27 1.27)) (justify left bottom))
   )
@@
   )
   (text "Power" (at 84.455 92.71 0)
+    (effects (font (size 1.27 1.27)) (justify left bottom))
+  )
+  (text "JC" (at 50.8 38.735 0)
     (effects (font (size 1.27 1.27)) (justify left bottom))
   )
@@
     (effects (font (size 1.27 1.27)) (justify left bottom))
   )
+  (text "JX" (at 41.275 39.37 0)
+    (effects (font (size 1.27 1.27)) (justify left bottom))
+  )

Commit message: cleanup
Other:
- note added: "Battery charging circuit"
Changed lines of the file:
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@@
     (effects (font (size 1.27 1.27)) (justify left bottom))
+  )
+  (text "Battery charging circuit" (at 92.075 113.03 0)
+    (effects (font (size 1 1)) (justify left bottom))
   )
   (text "Processing" (at 144.145 15.875 0)
