File: Tiny Handheld V2.1/Tiny handheld.kicad_pcb (KiCad board)
At the start: 2 copper layers, 34.3 x 58.4 mm, 44 parts, among them IC1 BQ21040DBVR, J1 VDisplay/prog1, J2 HDisplay/prog, J3 USB_C_Receptacle_USB2.0, U1 ATtiny85-20P, U2 ATtiny85-20S

Commit message: added JY JX and JC to schematic
Other:
- board text added: "TO DO:"
- board text removed: "TO DO: fix silkscreen error on com port (MISO / MOSI)"
Changed lines of the file:
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@@
     (effects (font (size 1.5 1.5) (thickness 0.2)))
   )
-  (gr_text "TO DO:\nfix silkscreen error on com port (MISO / MOSI)" (at 164 36.25) (layer "F.SilkS")
+  (gr_text "TO DO:\n" (at 164 36.25) (layer "F.SilkS")
     (effects (font (size 1.5 1.5) (thickness 0.3)))
   )

Commit message: Added games and potential oled driver
Oled drivers need to be implemented
Other:
- board text removed: "TO DO:"
Changed lines of the file:
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@@
     (effects (font (size 1.5 1.5) (thickness 0.2)))
-  )
-  (gr_text "TO DO:\n" (at 164 36.25) (layer "F.SilkS")
-    (effects (font (size 1.5 1.5) (thickness 0.3)))
   )
   (gr_text "PB5" (at 118.4 38.2 90) (layer "F.SilkS")
